File: _ PCB/Engine_Doctor_v0.1/Engine_Doctor_v0.1.sch (KiCad schematic (older format))
At the start: 7 parts, among them J1 Thermocouple, J2 BME280, J3 Battery, J4 Spare2, J5 Spare1, SW1 Power Switch, U1 lolin32_lite_V1.00

Commit message: PCB completed
Parts:
- J2: footprint Connector_PinHeader_2.54mm:PinHeader_1x04_P2.54mm_Vertical -> Connector_PinHeader_2.54mm:PinHeader_1x05_P2.54mm_Vertical
Changed lines of the file:
@@
 F 0 "J2" H 7978 5626 50  0000 L CNN
 F 1 "BME280" H 7978 5535 50  0000 L CNN
-F 2 "Connector_PinHeader_2.54mm:PinHeader_1x04_P2.54mm_Vertical" H 7950 5650 50  0001 C CNN
+F 2 "Connector_PinHeader_2.54mm:PinHeader_1x05_P2.54mm_Vertical" H 7950 5650 50  0001 C CNN
 F 3 "~" H 7950 5650 50  0001 C CNN
 	1    7950 5650
